File: secondarypower.sch (KiCad schematic (older format))
At the start: 4 parts, among them J5 Conn_01x02, U1 STM32F413RHTx

Commit message: Adds programming pins, bypass capacitors, & op amp
VoltageDivision.sch now uses OPA2990 to attenuate the supplemental battery signal by ~4. Timing crystal, NRST, bypass capacitors, & SWDIO & SWCLK connections added in.
Parts:
- removed J5: Conn_01x02, symbol Connector_Generic:Conn_01x02
- removed R10: 1k, symbol Device:R
- removed R9: 2k, symbol Device:R
- added C12, C13, C14, C16, C17, C18: 0.1u, Capacitor_SMD:C_0805_2012Metric, symbol Device:C
- added C15: 1u, Capacitor_SMD:C_0805_2012Metric, symbol Device:C
- added C19: 4.7u, Capacitor_SMD:C_0805_2012Metric, symbol Device:C
- added C20, C21: 8p, Capacitor_SMD:C_0805_2012Metric, symbol Device:C
- added C22: 2.2u, Capacitor_SMD:C_0805_2012Metric, symbol Device:C
- added H1, H2, H3, H4: MountingHole, MountingHole:MountingHole_3mm, symbol Mechanical:MountingHole
- added J4: Conn_01x04, Connector_Molex:Molex_Micro-Fit_3.0_43650-0400_1x04_P3.00mm_Horizontal, symbol Connector_Generic:Conn_01x04
- added SW1: SW_Push, Button_Switch_SMD:SW_SPST_B3SL-1002P, symbol Switch:SW_Push
- added Y1: 8M, Crystal:Crystal_SMD_TXC_7A-2Pin_5x3.2mm, symbol Device:Crystal
Connections:
- net labels added: NRST, SWCLK, SWDIO
- net labels removed: +12V
- wire segments 29 -> 83
- no-connect marks 0 -> 45
Other:
- note removed: "This 12V is \nfrom the supplementary\nbatteries\n"
