File: VoltageDivision.sch (KiCad schematic (older format))
At the start: 7 parts, among them J4 Conn_01x02, U4 TPS3711

Commit message: Adds programming pins, bypass capacitors, & op amp
VoltageDivision.sch now uses OPA2990 to attenuate the supplemental battery signal by ~4. Timing crystal, NRST, bypass capacitors, & SWDIO & SWCLK connections added in.
Parts:
- removed C12: 0.01uF, symbol Device:C
- removed J4: Conn_01x02, symbol Connector_Generic:Conn_01x02
- removed R8: 100, symbol Device:R
- removed U4: TPS3711, Package_TO_SOT_SMD:TSOT-23-6, symbol utsvt-chips:TPS3711
- added J5: Conn_01x02, Connector_Molex:Molex_Micro-Fit_3.0_43650-0200_1x02_P3.00mm_Horizontal, symbol Connector_Generic:Conn_01x02
- added U4: OPA2990, Package_TO_SOT_SMD:SOT-23, symbol utsvt-chips:OPA2990
- R5: value 1k -> 40k; footprint (none) -> Resistor_SMD:R_0805_2012Metric
- R6: value 1k -> 10k; footprint (none) -> Resistor_SMD:R_0805_2012Metric
- R7: value 100k -> 10k; footprint (none) -> Resistor_SMD:R_0805_2012Metric
Connections:
- net labels added: +15V, -15V
- net labels removed: +3.3V
- wire segments 29 -> 17
Other:
- note added: "This +12V is from the secondary\ndist. batteries.\n"
- note removed: "This 12V is \nfrom the supplementary\nbatteries\n"

Commit message: Added power flags
Connections:
- wire segments 17 -> 19
Changed lines of the file:
@@
 $EndComp
 Wire Wire Line
-	3250 2600 3250 2200
+	3250 2600 3250 2250
 Text Notes 3450 1950 2    50   ~ 0
 This +12V is from the secondary\ndist. batteries.\n
@@
 Wire Wire Line
 	4250 2600 4950 2600
+$Comp
+L power:PWR_FLAG #FLG0101
+U 1 1 5FC4A1C5
+P 4600 2350
+F 0 "#FLG0101" H 4600 2425 50  0001 C CNN
+F 1 "PWR_FLAG" V 4600 2477 50  0000 L CNN
+F 2 "" H 4600 2350 50  0001 C CNN
+F 3 "~" H 4600 2350 50  0001 C CNN
+	1    4600 2350
+	0    -1   -1   0
+$EndComp
+Connection ~ 4600 2350
+$Comp
+L power:PWR_FLAG #FLG0102
+U 1 1 5FC4AA40
+P 5900 2250
+F 0 "#FLG0102" H 5900 2325 50  0001 C CNN
+F 1 "PWR_FLAG" V 5900 2378 50  0000 L CNN
+F 2 "" H 5900 2250 50  0001 C CNN
+F 3 "~" H 5900 2250 50  0001 C CNN
+	1    5900 2250
+	0    1    1    0
+$EndComp
+Connection ~ 5900 2250
+$Comp
+L power:PWR_FLAG #FLG0103
+U 1 1 5FC4AB8B
+P 3250 2250
+F 0 "#FLG0103" H 3250 2325 50  0001 C CNN
+F 1 "PWR_FLAG" V 3250 2378 50  0000 L CNN
+F 2 "" H 3250 2250 50  0001 C CNN
+F 3 "~" H 3250 2250 50  0001 C CNN
+	1    3250 2250
+	0    1    1    0
+$EndComp
+Connection ~ 3250 2250
+Wire Wire Line
+	3250 2250 3250 2200
+Wire Wire Line
+	5750 3050 5750 3200
 $EndSCHEMATC
