File: CAN.sch (KiCad schematic (older format))
At the start: 20 parts, among them J1 CAN_Out, J2 CAN_Out, U2 ADM3055E, U3 CDSOT23-T24CAN

Commit message: Lays out schematic and PCB of v1.0
Parts:
- removed JP1: Termination Resistors, Connector_PinHeader_2.54mm:PinHeader_1x02_P2.54mm_Horizontal, symbol Device:Jumper_NC_Small
- removed R3: 60, Resistor_SMD:R_0805_2012Metric, symbol Device:R
- J2: renamed from J1; footprint Connector_Molex:Molex_Micro-Fit_3.0_43650-0400_1x04_P3.00mm_Horizontal -> UTSVT_Connectors:Molex_MicroFit3.0_1x4xP3.00mm_PolarizingPeg_Vertical; symbol BPSMaster-rescue:CANConnector-utsvt-connectors -> utsvt-connectors:CANConnector
- J3: renamed from J2; footprint Connector_Molex:Molex_Micro-Fit_3.0_43650-0400_1x04_P3.00mm_Horizontal -> UTSVT_Connectors:Molex_MicroFit3.0_1x4xP3.00mm_PolarizingPeg_Vertical; symbol BPSMaster-rescue:CANConnector-utsvt-connectors -> utsvt-connectors:CANConnector
- R2: value 60 -> 120
- U2: symbol BPSMaster-rescue:ADM3055E-utsvt-chips -> utsvt-chips:ADM3055E
- renumbered C1 to C12, C2 to C13, C3 to C14, C4 to C15, C5 to C16, C6 to C17, C7 to C18, C8 to C19
Connections:
- net labels removed: TERM_H, TERM_L
- wire segments 120 -> 119
Other:
- note added: "CAN"
- moved on the sheet: C12, C13, C14, C15, C16, C17, C18, C19, L1, L2, R1, R2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
