File: Power-SupplementalMonitoringPCB.kicad_pcb (KiCad board)
At the start: 2 copper layers, 67.5 x 44.5 mm, 64 parts, among them J1 SWD, J2 CAN_Out, J3 CAN_Out, J4 PowerConn, J5 SuppPowerConnector, SW1 Reset, U1 STM32F413RHTx, U2 ADM3055E, U3 CDSOT23-T24CAN, U4 RI3-1205S, U5 NCP1117-3.3_SOT223, U6 RI3-1215S, U7 OPAx192-Q1, Y1 8M

Commit message: added UTSVT-KiCADLibraries as a submodule, updated PCB and main schematic to KiCAD 7.0
Other:
- net class Default removed
