File: SupplementalMonitoringBoard/current.kicad_sch (KiCad schematic)
At the start: 8 parts, among them U2 OPA842xDBV

Commit message: Supplemental MOnitoring Board
Parts:
- CC1: value .1uF -> 1nF; P/N (none) -> C0805C102J5HACAUTO
- CC2: P/N (none) -> UMK212ABJ225KG-T
- R1: P/N (none) -> CRCW080510K0FKEAC
- R14: value 150K -> 150k; P/N (none) -> 0805W8F1503T5E
- R2: value 50K -> 50k; P/N (none) -> PNM0805E5002BST1
- R4: value 10K -> 10k; P/N (none) -> CRCW080510K0FKEAC
- R9: P/N (none) -> RCWE0805R100FNEA
- U2: P/N (none) -> SBOS267D
Connections:
- net +BATT renamed +12V
Changed lines of the file:
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@@
 	(paper "A4")
+	(junction
+		(at 72.39 90.17)
+		(diameter 0)
+		(color 0 0 0 0)
+	)
 	(junction
 		(at 97.79 90.17)
@@
 	(junction
 		(at 149.86 92.71)
-		(diameter 0)
-		(color 0 0 0 0)
-	)
-	(junction
-		(at 72.39 90.17)
 		(diameter 0)
 		(color 0 0 0 0)
@@
 	)
 	(symbol
+		(lib_id "power:+12V")
+		(at 72.39 90.17 0)
+		(unit 1)
+		(exclude_from_sim no)
+		(in_bom yes)
+		(on_board yes)
+		(dnp no)
+		(fields_autoplaced yes)
+		(property "Reference" "#PWR02"
+			(at 72.39 93.98 0)
+			(effects
+				(font
+					(size 1.27 1.27)
+				)
+				(hide yes)
+			)
+		)
+		(property "Value" "+12V"
+			(at 72.39 85.09 0)
+			(effects
+				(font
+					(size 1.27 1.27)
+				)
+			)
+		)
+		(property "Footprint" ""
+			(at 72.39 90.17 0)
+			(effects
+				(font
+					(size 1.27 1.27)
+				)
+				(hide yes)
+			)
+		)
+		(property "Datasheet" ""
+			(at 72.39 90.17 0)
+			(effects
+				(font
+					(size 1.27 1.27)
+				)
+				(hide yes)
+			)
+		)
+		(property "Description" "Power symbol creates a global label with name \"+12V\""
+			(at 72.39 90.17 0)
+			(effects
+				(font
+					(size 1.27 1.27)
+				)
+				(hide yes)
+			)
+		)
+		(pin "1"
+		)
+		(instances
+			(project "SupplementalMonitoringBoard"
+				(path "/aa0415d0-3287-4bc4-9a8e-766ada9ace2f/1e74c2bc-637a-422a-831e-fab1291cbb0a"
+					(reference "#PWR02")
+					(unit 1)
+				)
+			)
+		)
+	)
+	(symbol
 		(lib_id "Amplifier_Operational:OPA842xDBV")
 		(at 140.97 92.71 0)
@@
 			)
 		)
+		(property "P/N" "SBOS267D"
+			(at 140.97 92.71 0)
+			(effects
+				(font
+					(size 1.27 1.27)
+				)
+				(hide yes)
+			)
+		)
 		(pin "2"
 		)
@@
 			)
 		)
-		(property "Datasheet" "~"
+		(property "Datasheet" "https://www.mouser.com/datasheet/2/447/PYu_RT_1_to_0_01_RoHS_L_15-3461507.pdf"
 			(at 97.79 93.98 0)
 			(effects
@@
 			)
 		)
+		(property "P/N" "CRCW080510K0FKEAC"
+			(at 97.79 93.98 0)
+			(effects
+				(font
+					(size 1.27 1.27)
+				)
+				(hide yes)
+			)
+		)
 		(pin "1"
 		)
@@
 			)
 		)
-		(property "Datasheet" "~"
+		(property "Datasheet" "https://www.mouser.com/ProductDetail/Murata-Electronics/GRM219R6YA475KA73D?qs=eeBpzGFlv%252B%252Bho6epIC%2FPCA%3D%3D"
 			(at 195.58 129.54 0)
 			(effects
@@
 			)
 		)
+		(property "P/N" "UMK212ABJ225KG-T"
+			(at 195.58 129.54 0)
+			(effects
+				(font
+					(size 1.27 1.27)
+				)
+				(hide yes)
+			)
+		)
 		(pin "1"
 		)
@@
 			)
 		)
-		(property "Value" "150K"
+		(property "Value" "150k"
 			(at 124.46 102.87 90)
 			(effects
@@
 			)
 		)
-		(property "Datasheet" "~"
+		(property "Datasheet" "https://www.mouser.com/datasheet/2/1365/1-3044649.pdf"
 			(at 124.46 106.68 0)
 			(effects
@@
 			)
 		)
+		(property "P/N" "0805W8F1503T5E"
+			(at 124.46 106.68 0)
+			(effects
+				(font
+					(size 1.27 1.27)
+				)
+				(hide yes)
+			)
+		)
 		(pin "1"
 		)
@@
 			)
 		)
-		(property "Datasheet" "~"
+		(property "Datasheet" "https://www.vishay.com/docs/20019/rcwe.pdf"
 			(at 120.65 90.17 0)
 			(effects
@@
 			)
 		)
+		(property "P/N" "RCWE0805R100FNEA"
+			(at 120.65 90.17 0)
+			(effects
+				(font
+					(size 1.27 1.27)
+				)
+				(hide yes)
+			)
+		)
 		(pin "1"
 		)
@@
 				(path "/aa0415d0-3287-4bc4-9a8e-766ada9ace2f/1e74c2bc-637a-422a-831e-fab1291cbb0a"
 					(reference "R9")
-					(unit 1)
-				)
-			)
-		)
-	)
-	(symbol
-		(lib_id "power:+BATT")
-		(at 72.39 90.17 0)
-		(unit 1)
-		(exclude_from_sim no)
-		(in_bom yes)
-		(on_board yes)
-		(dnp no)
-		(fields_autoplaced yes)
-		(property "Reference" "#PWR02"
-			(at 72.39 93.98 0)
-			(effects
-				(font
-					(size 1.27 1.27)
-				)
-				(hide yes)
-			)
-		)
-		(property "Value" "+BATT"
-			(at 72.39 85.09 0)
-			(effects
-				(font
-					(size 1.27 1.27)
-				)
-			)
-		)
-		(property "Footprint" ""
-			(at 72.39 90.17 0)
-			(effects
-				(font
-					(size 1.27 1.27)
-				)
-				(hide yes)
-			)
-		)
-		(property "Datasheet" ""
-			(at 72.39 90.17 0)
-			(effects
-				(font
-					(size 1.27 1.27)
-				)
-				(hide yes)
-			)
-		)
-		(property "Description" "Power symbol creates a global label with name \"+BATT\""
-			(at 72.39 90.17 0)
-			(effects
-				(font
-					(size 1.27 1.27)
-				)
-				(hide yes)
-			)
-		)
-		(pin "1"
-		)
-		(instances
-			(project "SupplementalMonitoringBoard"
-				(path "/aa0415d0-3287-4bc4-9a8e-766ada9ace2f/1e74c2bc-637a-422a-831e-fab1291cbb0a"
-					(reference "#PWR02")
 					(unit 1)
 				)
@@
 			)
 		)
-		(property "Value" ".1uF"
+		(property "Value" "1nF"
 			(at 182.88 130.8162 0)
 			(effects
@@
 			)
 		)
-		(property "Datasheet" "~"
+		(property "Datasheet" "https://www.mouser.com/ProductDetail/KEMET/C0805C102J5HACAUTO?qs=j%252B1pi9TdxUbgwPgoM1tuTw%3D%3D"
 			(at 180.34 129.54 0)
 			(effects
@@
 			)
 		)
+		(property "P/N" "C0805C102J5HACAUTO"
+			(at 180.34 129.54 0)
+			(effects
+				(font
+					(size 1.27 1.27)
+				)
+				(hide yes)
+			)
+		)
 		(pin "1"
 		)
@@
 			)
 		)
-		(property "Value" "10K"
+		(property "Value" "10k"
 			(at 146.05 102.87 90)
 			(effects
@@
 			)
 		)
-		(property "Datasheet" "~"
+		(property "Datasheet" "https://www.mouser.com/datasheet/2/447/PYu_RT_1_to_0_01_RoHS_L_15-3461507.pdf"
 			(at 146.05 106.68 0)
 			(effects
@@
 			)
 		)
+		(property "P/N" "CRCW080510K0FKEAC"
+			(at 146.05 106.68 0)
+			(effects
+				(font
+					(size 1.27 1.27)
+				)
+				(hide yes)
+			)
+		)
 		(pin "1"
 		)
@@
 			)
 		)
-		(property "Value" "50K"
+		(property "Value" "50k"
 			(at 88.9 86.36 90)
 			(effects
@@
 			)
 		)
-		(property "Datasheet" "~"
+		(property "Datasheet" "https://www.vishay.com/docs/60057/pnm.pdf"
 			(at 88.9 90.17 0)
 			(effects
@@
 			(at 88.9 90.17 0)
 			(effects
+				(font
+					(size 1.27 1.27)
+				)
+				(hide yes)
+			)
+		)
+		(property "P/N" "PNM0805E5002BST1"
+			(at 88.9 90.17 0)
+			(effects

Commit message: Supplemental Monitoring Board
Parts:
- R1, R4: P/N CRCW080510K0FKEAC -> RT0603FRE0710KL
- R14: P/N 0805W8F1503T5E -> ERJ-UP6D1503V
- R2: P/N PNM0805E5002BST1 -> PTN0805E5002BST1
- R9: P/N RCWE0805R100FNEA -> WSLP0805R0100DEA
Changed lines of the file:
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@@
 			)
 		)
-		(property "Datasheet" "https://www.mouser.com/datasheet/2/447/PYu_RT_1_to_0_01_RoHS_L_15-3461507.pdf"
+		(property "Datasheet" "https://www.mouser.com/ProductDetail/603-RT0603FRE0710KL"
 			(at 97.79 93.98 0)
 			(effects
@@
 			)
 		)
-		(property "P/N" "CRCW080510K0FKEAC"
+		(property "P/N" "RT0603FRE0710KL "
 			(at 97.79 93.98 0)
 			(effects
@@
 			)
 		)
-		(property "Datasheet" "https://www.mouser.com/datasheet/2/1365/1-3044649.pdf"
+		(property "Datasheet" "https://www.mouser.com/catalog/specsheets/Panasonic_03-31-2024_Resistor_Anti-Sulfur(ERJ-UP6D-Series).pdf"
 			(at 124.46 106.68 0)
 			(effects
@@
 			)
 		)
-		(property "P/N" "0805W8F1503T5E"
+		(property "P/N" "ERJ-UP6D1503V "
 			(at 124.46 106.68 0)
 			(effects
@@
 			)
 		)
-		(property "Datasheet" "https://www.vishay.com/docs/20019/rcwe.pdf"
+		(property "Datasheet" "https://www.vishay.com/docs/30122/wslp.pdf"
 			(at 120.65 90.17 0)
 			(effects
@@
 			)
 		)
-		(property "P/N" "RCWE0805R100FNEA"
+		(property "P/N" "WSLP0805R0100DEA "
 			(at 120.65 90.17 0)
 			(effects
@@
 			)
 		)
-		(property "Datasheet" "https://www.mouser.com/datasheet/2/447/PYu_RT_1_to_0_01_RoHS_L_15-3461507.pdf"
+		(property "Datasheet" "https://www.mouser.com/ProductDetail/603-RT0603FRE0710KL"
 			(at 146.05 106.68 0)
 			(effects
@@
 			)
 		)
-		(property "P/N" "CRCW080510K0FKEAC"
+		(property "P/N" "RT0603FRE0710KL "
 			(at 146.05 106.68 0)
 			(effects
@@
 			)
 		)
-		(property "Datasheet" "https://www.vishay.com/docs/60057/pnm.pdf"
+		(property "Datasheet" "https://www.vishay.com/docs/60026/ptn.pdf"
 			(at 88.9 90.17 0)
 			(effects
@@
 			)
 		)
-		(property "P/N" "PNM0805E5002BST1"
+		(property "P/N" "PTN0805E5002BST1"
 			(at 88.9 90.17 0)
 			(effects
